File: Hardware/MAX11609EEE-Breakout-Board-doubleHeaders.sch (EAGLE design)
At the start: 5 parts, among them U1 MAX11609EEE+

Commit message: These are the files that were sent to OSHPARK
Parts:
- removed JP3: (no value), pinhead:PINHD-1X13
- added JP2, JP4: (no value), pinhead:PINHD-1X7
Connections:
- net AIN0: now also JP2.5; no longer JP3.5
- net AIN1: now also JP2.6; no longer JP3.6
- net AIN2: now also JP2.7; no longer JP3.7
- net AIN3: now also JP4.1; no longer JP3.8
- net AIN4: now also JP4.2; no longer JP3.9
- net AIN5: now also JP4.3; no longer JP3.10
- net AIN6: now also JP4.4; no longer JP3.11
- net AIN7: now also JP4.5; no longer JP3.12
- net GND: now also JP2.2; no longer JP3.2
- net REF: now also JP4.6; no longer JP3.13
- net SCL: now also JP2.4; no longer JP3.4
- net SDA: now also JP2.3; no longer JP3.3
- net VDD: now also JP2.1; no longer JP3.1
Changed lines of the file:
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@@
 <part name="VDD4" library="supply1" deviceset="VDD" device=""/>
 <part name="PE3" library="supply1" deviceset="PE" device="" value="GND"/>
-<part name="JP3" library="pinhead" deviceset="PINHD-1X13" device=""/>
+<part name="JP2" library="pinhead" deviceset="PINHD-1X7" device=""/>
+<part name="JP4" library="pinhead" deviceset="PINHD-1X7" device=""/>
 </parts>
 <sheets>
@@
 <instance part="VDD4" gate="G$1" x="111.76" y="38.1"/>
 <instance part="PE3" gate="M" x="111.76" y="17.78"/>
-<instance part="JP3" gate="A" x="147.32" y="30.48"/>
+<instance part="JP2" gate="A" x="147.32" y="38.1"/>
+<instance part="JP4" gate="A" x="147.32" y="12.7"/>
 </instances>
 <busses>
@@
 </segment>
 <segment>
-<pinref part="JP3" gate="A" pin="3"/>
 <wire x1="144.78" y1="40.64" x2="134.62" y2="40.64" width="0.1524" layer="91"/>
 <label x="134.62" y="40.64" size="1.778" layer="95"/>
+<pinref part="JP2" gate="A" pin="3"/>
 </segment>
 </net>
@@
 </segment>
 <segment>
-<pinref part="JP3" gate="A" pin="4"/>
 <wire x1="144.78" y1="38.1" x2="134.62" y2="38.1" width="0.1524" layer="91"/>
 <label x="134.62" y="38.1" size="1.778" layer="95"/>
+<pinref part="JP2" gate="A" pin="4"/>
 </segment>
 </net>
@@
 </segment>
 <segment>
-<pinref part="JP3" gate="A" pin="1"/>
 <wire x1="144.78" y1="45.72" x2="134.62" y2="45.72" width="0.1524" layer="91"/>
 <label x="134.62" y="45.72" size="1.778" layer="95"/>
+<pinref part="JP2" gate="A" pin="1"/>
 </segment>
 </net>
@@
 </segment>
 <segment>
-<pinref part="JP3" gate="A" pin="12"/>
-<wire x1="144.78" y1="17.78" x2="134.62" y2="17.78" width="0.1524" layer="91"/>
-<label x="134.62" y="17.78" size="1.778" layer="95"/>
+<wire x1="144.78" y1="10.16" x2="134.62" y2="10.16" width="0.1524" layer="91"/>
+<label x="134.62" y="10.16" size="1.778" layer="95"/>
+<pinref part="JP4" gate="A" pin="5"/>
 </segment>
 </net>
@@
 </segment>
 <segment>
-<pinref part="JP3" gate="A" pin="11"/>
-<wire x1="144.78" y1="20.32" x2="134.62" y2="20.32" width="0.1524" layer="91"/>
-<label x="134.62" y="20.32" size="1.778" layer="95"/>
+<wire x1="144.78" y1="12.7" x2="134.62" y2="12.7" width="0.1524" layer="91"/>
+<label x="134.62" y="12.7" size="1.778" layer="95"/>
+<pinref part="JP4" gate="A" pin="4"/>
 </segment>
 </net>
@@
 </segment>
 <segment>
-<pinref part="JP3" gate="A" pin="10"/>
-<wire x1="144.78" y1="22.86" x2="134.62" y2="22.86" width="0.1524" layer="91"/>
-<label x="134.62" y="22.86" size="1.778" layer="95"/>
+<wire x1="144.78" y1="15.24" x2="134.62" y2="15.24" width="0.1524" layer="91"/>
+<label x="134.62" y="15.24" size="1.778" layer="95"/>
+<pinref part="JP4" gate="A" pin="3"/>
 </segment>
 </net>
@@
 </segment>
 <segment>
-<pinref part="JP3" gate="A" pin="9"/>
-<wire x1="144.78" y1="25.4" x2="134.62" y2="25.4" width="0.1524" layer="91"/>
-<label x="134.62" y="25.4" size="1.778" layer="95"/>
+<wire x1="144.78" y1="17.78" x2="134.62" y2="17.78" width="0.1524" layer="91"/>
+<label x="134.62" y="17.78" size="1.778" layer="95"/>
+<pinref part="JP4" gate="A" pin="2"/>
 </segment>
 </net>
@@
 </segment>
 <segment>
-<pinref part="JP3" gate="A" pin="5"/>
 <wire x1="144.78" y1="35.56" x2="134.62" y2="35.56" width="0.1524" layer="91"/>
 <label x="134.62" y="35.56" size="1.778" layer="95"/>
+<pinref part="JP2" gate="A" pin="5"/>
 </segment>
 </net>
@@
 </segment>
 <segment>
-<pinref part="JP3" gate="A" pin="6"/>
 <wire x1="144.78" y1="33.02" x2="134.62" y2="33.02" width="0.1524" layer="91"/>
 <label x="134.62" y="33.02" size="1.778" layer="95"/>
+<pinref part="JP2" gate="A" pin="6"/>
 </segment>
 </net>
@@
 </segment>
 <segment>
-<pinref part="JP3" gate="A" pin="7"/>
 <wire x1="144.78" y1="30.48" x2="134.62" y2="30.48" width="0.1524" layer="91"/>
 <label x="134.62" y="30.48" size="1.778" layer="95"/>
+<pinref part="JP2" gate="A" pin="7"/>
 </segment>
 </net>
@@
 </segment>
 <segment>
-<pinref part="JP3" gate="A" pin="8"/>
-<wire x1="144.78" y1="27.94" x2="134.62" y2="27.94" width="0.1524" layer="91"/>
-<label x="134.62" y="27.94" size="1.778" layer="95"/>
+<wire x1="144.78" y1="20.32" x2="134.62" y2="20.32" width="0.1524" layer="91"/>
+<label x="134.62" y="20.32" size="1.778" layer="95"/>
+<pinref part="JP4" gate="A" pin="1"/>
 </segment>
 </net>
@@
 </segment>
 <segment>
-<pinref part="JP3" gate="A" pin="13"/>
-<wire x1="144.78" y1="15.24" x2="134.62" y2="15.24" width="0.1524" layer="91"/>
-<label x="134.62" y="15.24" size="1.778" layer="95"/>
+<wire x1="144.78" y1="7.62" x2="134.62" y2="7.62" width="0.1524" layer="91"/>
+<label x="134.62" y="7.62" size="1.778" layer="95"/>
+<pinref part="JP4" gate="A" pin="6"/>
 </segment>
 </net>
 <net name="GND" class="0">
 <segment>
-<pinref part="JP3" gate="A" pin="2"/>
 <wire x1="144.78" y1="43.18" x2="134.62" y2="43.18" width="0.1524" layer="91"/>
 <label x="134.62" y="43.18" size="1.778" layer="95"/>
-</segment>
-<segment>
+<pinref part="JP2" gate="A" pin="2"/>
+</segment>
+<segment>
